File: LocalElectricCircuit.sch (EAGLE design)
At the start: 46 parts, among them IC1 PIC32MX360F512L, J1 Prog. Port, J3 Prog. Port, T1 PN100, U1 ADS1118, U2 ADS1118

Commit message: Fan out step numero uno
Parts:
- removed PIC32_POWER_EN: (no value), pinhead:PINHD-1X2
Connections:
- net +3V3: no longer PIC32_POWER_EN.1, PIC32_POWER_EN.2
Changed lines of the file:
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@@
 <part name="R14" library="rcl" deviceset="R-US_" device="M1206" value="50"/>
 <part name="PIC16_POWER_EN" library="pinhead" deviceset="PINHD-1X2" device=""/>
-<part name="PIC32_POWER_EN" library="pinhead" deviceset="PINHD-1X2" device=""/>
 <part name="R15" library="rcl" deviceset="R-US_" device="0309/12" value="1k"/>
 </parts>
@@
 <instance part="R14" gate="G$1" x="203.2" y="81.28" rot="R180"/>
 <instance part="PIC16_POWER_EN" gate="G$1" x="289.56" y="30.48"/>
-<instance part="PIC32_POWER_EN" gate="G$1" x="101.6" y="167.64"/>
 <instance part="R15" gate="G$1" x="200.66" y="-30.48" rot="R180"/>
 </instances>
@@
 </segment>
 <segment>
-<pinref part="PIC32_POWER_EN" gate="G$1" pin="2"/>
 <wire x1="99.06" y1="167.64" x2="93.98" y2="167.64" width="0.1524" layer="91"/>
-<label x="93.98" y="167.64" size="1.778" layer="95" rot="R180"/>
 </segment>
 <segment>
@@
 </segment>
 <segment>
-<pinref part="PIC32_POWER_EN" gate="G$1" pin="1"/>
-<wire x1="99.06" y1="170.18" x2="93.98" y2="170.18" width="0.1524" layer="91"/>
-<label x="93.98" y="170.18" size="1.778" layer="95" rot="R180"/>
-</segment>
-<segment>

Commit message: Power plane progress
Parts:
- removed R10, R9: 1k, rcl:R-US_0309/12
- removed T1: PN100, transistor:2N3704
Connections:
- removed net CONDUCTIVITY_ENABLE_3V: IC1.RC3, R15.2
- removed net CONDUCTIVITY_ENABLE_5V: J2.C14, R10.2, R9.1
- removed net N$10: R15.1, T1.B
- removed net N$5: R9.2, T1.E
- new net CONDUCTIVITY_ENABLE: IC1.RC3, J2.C14, R15.2
- net +3V3: now also R15.1
- net +5V: no longer T1.C
- net GND_5V: no longer R10.1
Other:
- moved on the sheet: R15
Changed lines of the file:
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@@
 <setting verticaltext="up"/>
 </settings>
-<grid distance="0.1" unitdist="inch" unit="inch" style="lines" multiple="1" display="no" altdistance="0.01" altunitdist="inch" altunit="inch"/>
+<grid distance="0.1" unitdist="inch" unit="inch" style="lines" multiple="1" display="no" altdistance="0.025" altunitdist="inch" altunit="inch"/>
 <layers>
 <layer number="1" name="Top" color="4" fill="1" visible="no" active="no"/>
@@
 <part name="C10" library="resistor" deviceset="C-US" device="C1206" value="0.1uF"/>
 <part name="C11" library="resistor" deviceset="C-US" device="C1206" value="0.01uF"/>
-<part name="T1" library="transistor" deviceset="2N3704" device="" value="PN100"/>
 <part name="J3" library="con-amp" deviceset="520258-3" device="" value="Prog. Port"/>
 <part name="R7" library="rcl" deviceset="R-US_" device="M1206" value="50k"/>
@@
 <part name="R4" library="rcl" deviceset="R-US_" device="0309/12" value="1k"/>
 <part name="R8" library="rcl" deviceset="R-US_" device="0309/12" value="1k"/>
-<part name="R9" library="rcl" deviceset="R-US_" device="0309/12" value="1k"/>
-<part name="R10" library="rcl" deviceset="R-US_" device="0309/12" value="1k"/>
 <part name="R5" library="rcl" deviceset="R-US_" device="M1206" value="50"/>
 <part name="R6" library="rcl" deviceset="R-US_" device="M1206" value="50"/>
@@
 <instance part="C10" gate="G$1" x="231.14" y="25.4" rot="R90"/>
 <instance part="C11" gate="G$1" x="231.14" y="33.02" rot="R90"/>
-<instance part="T1" gate="G$1" x="208.28" y="-30.48"/>
 <instance part="J3" gate="G$1" x="292.1" y="5.08"/>
 <instance part="R7" gate="G$1" x="281.94" y="12.7" rot="R90"/>
@@
 <instance part="R4" gate="G$1" x="147.32" y="2.54" rot="R180"/>
 <instance part="R8" gate="G$1" x="139.7" y="-2.54" rot="R180"/>
-<instance part="R9" gate="G$1" x="210.82" y="-43.18" rot="R90"/>
-<instance part="R10" gate="G$1" x="210.82" y="-58.42" rot="R90"/>
 <instance part="R5" gate="G$1" x="248.92" y="119.38" rot="R180"/>
 <instance part="R6" gate="G$1" x="243.84" y="114.3" rot="R180"/>
@@
 <instance part="R14" gate="G$1" x="203.2" y="81.28" rot="R180"/>
 <instance part="PIC16_POWER_EN" gate="G$1" x="289.56" y="30.48"/>
-<instance part="R15" gate="G$1" x="200.66" y="-30.48" rot="R180"/>
+<instance part="R15" gate="G$1" x="231.14" y="-73.66" rot="R180"/>
 </instances>
 <busses>
@@
 <wire x1="76.2" y1="114.3" x2="76.2" y2="116.84" width="0.1524" layer="91"/>
 <label x="76.835" y="116.84" size="1.778" layer="95" rot="R90"/>
+</segment>
+<segment>
+<label x="241.935" y="-63.5" size="1.778" layer="95" rot="R90"/>
+<pinref part="R15" gate="G$1" pin="1"/>
+<wire x1="236.22" y1="-73.66" x2="241.3" y2="-73.66" width="0.1524" layer="91"/>
+<wire x1="241.3" y1="-73.66" x2="241.3" y2="-63.5" width="0.1524" layer="91"/>
 </segment>
 </net>
@@
 <label x="-55.88" y="155.575" size="1.778" layer="95" rot="R180"/>
 </segment>
-<segment>
-<label x="210.185" y="-66.04" size="1.778" layer="95" rot="R270"/>
-<pinref part="R10" gate="G$1" pin="1"/>
-<wire x1="210.82" y1="-66.04" x2="210.82" y2="-63.5" width="0.1524" layer="91"/>
-</segment>
 </net>
 <net name="+5V" class="1">
@@
 <wire x1="-45.72" y1="147.32" x2="-55.88" y2="147.32" width="0.1524" layer="91"/>
 <label x="-55.88" y="147.955" size="1.778" layer="95" rot="R180"/>
-</segment>
-<segment>
-<label x="211.455" y="-22.86" size="1.778" layer="95" rot="R90"/>
-<pinref part="T1" gate="G$1" pin="C"/>
-<wire x1="210.82" y1="-22.86" x2="210.82" y2="-25.4" width="0.1524" layer="91"/>
 </segment>
 </net>
@@
 </segment>
 </net>
-<net name="CONDUCTIVITY_ENABLE_5V" class="0">
-<segment>
-<label x="213.36" y="-51.435" size="1.778" layer="95"/>
-<wire x1="210.82" y1="-50.8" x2="213.36" y2="-50.8" width="0.1524" layer="91"/>
-<pinref part="R9" gate="G$1" pin="1"/>
-<pinref part="R10" gate="G$1" pin="2"/>
-<wire x1="210.82" y1="-48.26" x2="210.82" y2="-50.8" width="0.1524" layer="91"/>
-<junction x="210.82" y="-50.8"/>
-<wire x1="210.82" y1="-50.8" x2="210.82" y2="-53.34" width="0.1524" layer="91"/>
+<net name="CONDUCTIVITY_ENABLE" class="0">
+<segment>
+<label x="220.98" y="-73.025" size="1.778" layer="95" rot="R180"/>
+<pinref part="R15" gate="G$1" pin="2"/>
+<wire x1="220.98" y1="-73.66" x2="226.06" y2="-73.66" width="0.1524" layer="91"/>
+<wire x1="226.06" y1="-73.66" x2="226.06" y2="-83.82" width="0.1524" layer="91"/>
+<wire x1="226.06" y1="-83.82" x2="248.92" y2="-83.82" width="0.1524" layer="91"/>
+<junction x="226.06" y="-73.66"/>
+<label x="248.92" y="-84.455" size="1.778" layer="95"/>
+</segment>
+<segment>
+<pinref part="IC1" gate="G$1" pin="RC3"/>
+<wire x1="17.78" y1="73.66" x2="12.7" y2="73.66" width="0.1524" layer="91"/>
+<label x="12.7" y="74.295" size="1.778" layer="95" rot="R180"/>
 </segment>
 <segment>
@@
 </segment>
 </net>
-<net name="CONDUCTIVITY_ENABLE_3V" class="0">
-<segment>
-<label x="190.5" y="-29.845" size="1.778" layer="95" rot="R180"/>
-<pinref part="R15" gate="G$1" pin="2"/>
-<wire x1="190.5" y1="-30.48" x2="195.58" y2="-30.48" width="0.1524" layer="91"/>
-</segment>
-<segment>
-<pinref part="IC1" gate="G$1" pin="RC3"/>
-<wire x1="17.78" y1="73.66" x2="12.7" y2="73.66" width="0.1524" layer="91"/>
-<label x="12.7" y="74.295" size="1.778" layer="95" rot="R180"/>
-</segment>
-</net>
-<net name="N$5" class="0">
-<segment>
-<pinref part="R9" gate="G$1" pin="2"/>
-<pinref part="T1" gate="G$1" pin="E"/>
-<wire x1="210.82" y1="-38.1" x2="210.82" y2="-35.56" width="0.1524" layer="91"/>
-</segment>
-</net>
 <net name="N$1" class="0">
 <segment>
@@
 </segment>
 </net>
-<net name="N$10" class="0">
-<segment>
-<pinref part="R15" gate="G$1" pin="1"/>
-<pinref part="T1" gate="G$1" pin="B"/>
-</segment>
-</net>

Commit message: 👌
Other:
- note removed: "ToDo: -Figure out PIC pins for I2C -Figure out PIC pins for selector of conductivity (3 GPIO) -Pull up for 3V logic for conductivity -Figure out 11 analog pins for the PIC (Avaliable are: AN0,AN1,AN3-AN5,AN8-AN15) -Figure out PIC pins for 2 thermistor inputs -Figure out PIC pins for 3 eurocard temp inputs -Figure out PIC pins for 6 power supervision inputs -Figure out PIC pins for ballast (8 GPIO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"
Changed lines of the file:
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@@
 <setting verticaltext="up"/>
 </settings>
-<grid distance="0.1" unitdist="inch" unit="inch" style="lines" multiple="1" display="no" altdistance="0.025" altunitdist="inch" altunit="inch"/>
+<grid distance="0.1" unitdist="inch" unit="inch" style="lines" multiple="1" display="no" altdistance="0.01" altunitdist="inch" altunit="inch"/>
 <layers>
 <layer number="1" name="Top" color="4" fill="1" visible="no" active="no"/>
@@
 <sheet>
 <plain>
-<text x="297.18" y="121.92" size="3.556" layer="91" align="top-left">ToDo:
-   -Figure out PIC pins for I2C
-   -Figure out PIC pins for selector of conductivity (3 GPIO)
-   -Pull up for 3V logic for conductivity
-   -Figure out 11 analog pins for the PIC (Avaliable are: AN0,AN1,AN3-AN5,AN8-AN15)
-      -Figure out PIC pins for 2 thermistor inputs
-      -Figure out PIC pins for 3 eurocard temp inputs
-      -Figure out PIC pins for 6 power supervision inputs
-   -Figure out PIC pins for ballast (8 GPIO)
-   -Figure out what the oscillator is
-   -Make a PIC programming circuit
-</text>
 </plain>
 <instances>
@@
 </schematic>
 </drawing>
-<compatibility>
-<note version="6.3" minversion="6.2.2" severity="warning">
-Since Version 6.2.2 text objects can contain more than one line,
-which will not be processed correctly with this version.
-</note>
-</compatibility>
 </eagle>
