File: LocalElectricCircuit.brd (EAGLE design)
At the start: 160 x 100 mm, 53 parts, among them IC1 PIC32MX360F512L, U1 ADS1118, U2 ADS1118, X2 MALE_VGA

Commit message: Did a whole ton of stuff. Added the level-shifting hardware Added fan out for ADC's Worked on clearing some DRC errors ETC
Parts:
- added JP3, JP4, JP5, JP6: (no value), pinhead:1X05
- added R10, R17: 680, resistor:R1206
- added R16, R9: 510, resistor:R1206
- added V1, V2: 74125N, 74ttl-din:DIL14
- moved R6 147.8 mm to (198.8, -94.4)
- moved R5 145.7 mm to (198.8, -89.4)
- moved U1 141.9 mm to (206.8, -94.4)
- moved C9 141.9 mm to (204.0, -94.4)
- moved R11 124.0 mm to (198.8, -99.4), turned to 270 degrees
- moved R13 94.2 mm to (139.6, -94.4)
- moved R12 89.4 mm to (139.6, -89.4)
- moved C8 82.9 mm to (144.8, -94.4)
- moved U2 82.9 mm to (147.6, -94.4)
- moved R14 71.3 mm to (139.6, -99.4)
- moved R15 13.7 mm to (113.8, -1.60)
Connections:
- new net ADC1_DIN: JP3.5, R5.1, V1.6
- new net ADC1_DIVIDED: R10.2, R9.1, V1.9
- new net ADC1_DOUT: JP3.4, R6.1, R9.2
- new net ADC1_SCK: JP4.1, R11.2, V1.3
- new net ADC2_DIN: JP5.5, R12.1, V2.6
- new net ADC2_DIVIDED: R16.1, R17.2, V2.9
- new net ADC2_DOUT: JP5.4, R13.1, R16.2
- new net ADC2_SCK: JP6.1, R14.2, V2.3
- net +5V: now also JP3.3, JP5.3, V1.14, V2.14
- net GND: now also JP3.2, JP5.2
- net GND_5V: now also JP4.2, JP4.3, JP6.2, JP6.3, R10.1, R17.1, V1.1, V1.10, V1.11, V1.12, V1.13, V1.4, V1.7, V2.1, V2.10, V2.11, V2.12, V2.13, V2.4, V2.7
- net PROBE_DIFF_HOR: now also JP6.4
- net PROBE_DIFF_VERT: now also JP4.5
- net PROBE_HOR_1_RIGHT: now also JP3.1
- net PROBE_HOR_2_LEFT: now also JP5.1
- net PROBE_VERT_1_UP: now also JP4.4
- net PROBE_VERT_2_DOWN: now also JP6.5
- net SCK1: now also V1.2; no longer R11.2
- net SCK2: now also V2.2; no longer R14.2
- net SDI1: now also V1.8; no longer R6.1
- net SDI2: now also V2.8; no longer R13.1
- net SDO1: now also V1.5; no longer R5.1
- net SDO2: now also V2.5; no longer R12.1
- net U2RX: now also U$1.3; no longer U$1.4
- net U2TX: now also U$1.4; no longer U$1.3
Routing:
- net GND_5V: track 8.38 -> 43.0 mm, vias 0 -> 4
- net +5V: track 3.90 -> 21.7 mm, vias 0 -> 2
- net N$4: track 2.24 -> 11.8 mm, vias 0 -> 2
- net N$8: track 2.24 -> 11.8 mm, vias 0 -> 2
- net ADC2_DOUT: track 0.00 -> 8.73 mm
- net ADC1_DOUT: track 0.00 -> 8.73 mm
- net N$43: track 7.19 -> 0.00 mm
- net N$42: track 7.02 -> 0.00 mm
- net N$41: track 6.86 -> 0.00 mm
- net +3V3: track 112.2 -> 105.5 mm, vias 9 -> 8
- net N$38: track 6.69 -> 0.00 mm
- net N$37: track 6.53 -> 0.00 mm
- net N$34: track 6.36 -> 0.00 mm
- net N$33: track 6.19 -> 0.00 mm
- net GND: track 4.48 -> 10.3 mm, vias 0 -> 2
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
Commit message: Pre auto-route
Parts:
- removed R15, R4, R8: 1k, rcl:0309/12
- moved V1 112.4 mm to (98.9, -19.6), turned to 270 degrees
- moved C9 102.4 mm to (134.0, -19.6)
- moved R11 102.4 mm to (128.8, -24.6)
- moved R5 102.4 mm to (128.8, -14.6)
- moved R6 102.4 mm to (128.8, -19.6)
- moved U1 102.4 mm to (136.8, -19.6)
- moved JP3 102.4 mm to (136.8, -13.2)
- moved JP4 102.4 mm to (136.8, -25.9)
- moved V2 100.6 mm to (98.9, 1.80), turned to 270 degrees
- moved R10 98.2 mm to (106.9, -21.0), turned to 270 degrees
- moved C8 96.8 mm to (134.0, 1.80)
- moved JP5 96.8 mm to (136.8, 8.15)
- moved JP6 96.8 mm to (136.8, -4.55)
- moved R12 96.8 mm to (128.8, 6.80)
- moved R13 96.8 mm to (128.8, 1.80)
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Connections:
- new net PIC_COND_EN: IC1.8, V2.12
- net +3V3: no longer R15.1
- net CONDUCTIVITY_ENABLE: now also V2.11; no longer IC1.8, R15.2
- net EXT_TEMP: no longer R8.1
- net GND_3V3: no longer R4.2, R8.2
- net GND_5V: no longer V1.12, V2.11, V2.12
- net RB_TEMP: no longer R4.1
Routing:
- net OSC1: track 7.30 -> 24.1 mm
- net OSC2: track 6.67 -> 21.6 mm
- net N$126: track 8.39 -> 0.00 mm, vias 0 -> 1
- net N$114: track 8.39 -> 0.00 mm, vias 0 -> 1
- net N$200: track 8.39 -> 0.00 mm, vias 0 -> 1
- net N$211: track 8.39 -> 0.00 mm, vias 0 -> 1
- net N$124: track 8.06 -> 0.00 mm, vias 0 -> 1
- net N$58: track 8.06 -> 0.00 mm, vias 0 -> 1
- net N$209: track 8.06 -> 0.00 mm
- net N$239: track 8.06 -> 0.00 mm
- net N$110: track 7.73 -> 0.00 mm, vias 0 -> 1
- net N$122: track 7.73 -> 0.00 mm, vias 0 -> 1
- net N$197: track 7.73 -> 0.00 mm, vias 0 -> 1
- net N$207: track 7.73 -> 0.00 mm
- net CONDUCTIVITY_ENABLE: track 7.60 -> 0.00 mm, vias 1 -> 0
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
Commit message: Actually pre auto routing
Parts:
- moved R10 12.7 mm to (106.9, -33.7)
- moved C8 12.7 mm to (134.0, -10.9)
- moved R13 12.7 mm to (128.8, -10.9)
- moved R17 12.7 mm to (106.9, -12.3)
- moved R5 12.7 mm to (128.8, -27.3)
- moved U2 12.7 mm to (136.8, -10.9)
- moved V2 12.7 mm to (98.9, -10.9)
- moved JP3 12.7 mm to (136.8, -25.9)
- moved JP4 12.7 mm to (136.8, -38.6)
- moved JP5 12.7 mm to (136.8, -4.55)
- moved JP6 12.7 mm to (136.8, -17.2)
- moved R12 12.7 mm to (128.8, -5.90)
- moved R14 12.7 mm to (128.8, -15.9)
- moved R16 12.7 mm to (106.9, -17.5)
- moved R9 12.7 mm to (106.9, -38.9)
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Routing:
- net GND_3V3: track 108.9 -> 172.2 mm
- net +3V3: track 110.9 -> 174.2 mm
- net GND_5V: track 47.3 -> 90.7 mm
- net +5V: track 21.7 -> 62.6 mm
- added copper zone on layer 1, net +3V3
- added copper zone on layer 1, net +5V
- added copper zone on layer 16, net GND
- added copper zone on layer 16, net GND_3V3
- added copper zone on layer 16, net GND_5V
