File: MagAltBreakout.brd (EAGLE design)
At the start: 49.5 x 44.5 mm, 0 parts

Commit message: Bloon
Parts:
- added U$5: (no value), Logos:BALLOON
Changed lines of the file:
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@@
 </autorouter>
 <elements>
+<element name="U$5" library="Logos" package="BALLOON" value="" x="14.960071875" y="38.500721875" smashed="yes"/>
 </elements>
 <signals>
