File: DebugPowerSupplyBoard/DebugPowerSupplyBoard.brd (EAGLE design)
At the start: 160 x 100 mm, 281 parts, among them IC1 LD117AV33, IC2 7805T

Commit message: Alright, got it perfect, including adding a box around the board label ❤
Parts:
- moved U$6 3.59 mm to (30.2, 94.0)
- turned U$1 to 0 degrees
- turned U$10 to 0 degrees
- turned U$100 to 0 degrees
- turned U$101 to 0 degrees
- turned U$102 to 0 degrees
- turned U$103 to 0 degrees
- turned U$104 to 0 degrees
- turned U$105 to 0 degrees
- turned U$106 to 0 degrees
- turned U$107 to 0 degrees
- turned U$108 to 0 degrees
- turned U$109 to 0 degrees
- turned U$11 to 0 degrees
- turned U$110 to 0 degrees
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Routing:
- net GND: track 2259.9 -> 2261.4 mm

Commit message: Finished the board
Parts:
- removed U$1, U$10, U$100, U$101, U$102, U$103, U$104, U$105, U$106, U$107, U$108, U$109, U$11, U$110, U$111, U$112, U$113, U$114, U$115, U$116, U$117, U$118, U$119, U$12, U$120, U$121, U$122, U$123, U$124, U$125, U$126, U$127, U$128, U$129, U$13, U$130, U$131, U$132, U$133, U$134, U$135, U$136, U$137, U$138, U$139, U$14, U$140, U$141, U$142, U$143, U$144, U$145, U$146, U$147, U$148, U$149, U$15, U$150, U$151, U$152, U$153, U$154, U$155, U$156, U$157, U$158, U$159, U$16, U$160, U$161, U$162, U$163, U$164, U$165, U$166, U$167, U$168, U$169, U$17, U$170, U$171, U$172, U$173, U$174, U$175, U$176, U$177, U$178, U$179, U$18, U$180, U$181, U$182, U$183, U$184, U$185, U$186, U$187, U$188, U$189, U$19, U$190, U$191, U$192, U$193, U$194, U$195, U$196, U$197, U$198, U$199, U$2, U$20, U$200, U$201, U$202, U$203, U$204, U$205, U$206, U$207, U$208, U$209, U$210, U$211, U$212, U$213, U$214, U$215, U$216, U$217, U$218, U$219, U$22, U$220, U$221, U$222, U$223, U$224, U$225, U$226, U$227, U$228, U$229, U$23, U$230, U$231, U$232, U$233, U$234, U$235, U$236, U$237, U$238, U$239, U$24, U$240, U$241, U$242, U$243, U$244, U$245, U$246, U$247, U$248, U$249, U$25, U$250, U$251, U$252, U$253, U$254, U$255, U$256, U$257, U$258, U$259, U$26, U$260, U$261, U$262, U$263, U$264, U$265, U$266, U$267, U$268, U$269, U$27, U$270, U$271, U$272, U$28, U$29, U$3, U$30, U$31, U$32, U$33, U$34, U$35, U$36, U$37, U$38, U$39, U$4, U$40, U$41, U$42, U$43, U$44, U$45, U$46, U$47, U$48, U$49, U$5, U$50, U$51, U$52, U$53, U$54, U$55, U$56, U$57, U$58, U$59, U$60, U$61, U$62, U$63, U$64, U$65, U$66, U$67, U$68, U$69, U$7, U$70, U$71, U$72, U$73, U$74, U$75, U$76, U$77, U$78, U$79, U$8, U$80, U$81, U$82, U$83, U$84, U$85, U$86, U$87, U$88, U$89, U$9, U$90, U$91, U$92, U$93, U$94, U$95, U$96, U$97, U$98, U$99: (no value), Logos:BALLOON
- added U$21, U$273, U$274, U$275, U$276, U$277, U$278, U$279, U$280, U$281, U$282, U$283, U$284, U$285, U$286, U$287, U$288, U$289, U$290, U$291, U$292, U$293, U$294, U$295, U$296, U$297, U$298, U$299, U$300, U$301, U$302, U$303, U$304, U$305, U$306, U$307, U$308, U$309, U$310, U$311, U$312, U$313, U$314, U$315, U$316, U$317, U$318, U$319, U$320, U$321, U$322, U$323, U$324, U$325, U$326, U$327, U$328, U$329, U$330, U$331, U$332, U$333, U$334, U$335, U$336, U$337, U$338, U$339, U$340, U$341, U$342, U$343, U$344, U$345, U$346, U$347, U$348, U$349, U$350, U$351, U$352, U$353, U$354, U$355, U$356, U$357, U$358, U$359, U$360, U$361, U$362, U$363, U$364, U$365, U$366, U$367, U$368, U$369, U$370, U$371, U$372, U$373, U$374, U$375, U$376, U$377, U$378, U$379, U$380, U$381, U$382, U$383, U$384, U$385, U$386, U$387, U$388, U$389, U$390, U$391, U$392, U$393, U$394, U$395, U$396, U$397, U$398, U$399, U$400, U$401, U$402, U$403, U$404, U$405, U$406, U$407, U$408, U$409, U$410, U$411, U$412, U$413, U$414, U$415, U$416, U$417, U$418, U$419, U$420, U$421, U$422, U$423, U$424, U$425, U$426, U$427, U$428, U$429, U$430, U$431, U$432, U$433, U$434, U$435, U$436, U$437, U$438, U$439, U$440, U$441, U$442, U$443, U$444, U$445, U$446, U$447, U$448, U$449, U$450, U$451, U$452, U$453, U$454, U$455, U$456, U$457, U$458, U$459, U$460, U$461, U$462, U$463, U$464, U$465, U$466, U$467, U$468, U$469, U$470, U$471, U$472, U$473, U$474, U$475, U$476, U$477, U$478, U$479, U$480, U$481, U$482, U$483, U$484, U$485, U$486, U$487, U$488, U$489, U$490, U$491, U$492, U$493, U$494, U$495, U$496, U$497, U$498, U$499, U$500, U$501, U$502, U$503, U$504, U$505, U$506, U$507, U$508, U$509, U$510, U$511, U$512, U$513, U$514, U$515, U$516, U$517, U$518, U$519, U$520, U$521, U$522, U$523, U$524, U$525, U$526, U$527, U$528, U$529, U$530, U$531, U$532, U$533, U$534, U$535, U$536, U$537, U$538, U$539, U$540, U$541: (no value), Logos:BALLOON
- moved C1 0.27 mm to (44.2, 82.5)
- moved C2 0.27 mm to (51.8, 82.5)
- moved C3 0.27 mm to (64.5, 69.8)
- moved C4 0.27 mm to (70.8, 73.7)
- moved C5 0.27 mm to (59.4, 82.5)
- moved C6 0.27 mm to (67.0, 82.5)
- moved IC1 0.27 mm to (34.0, 81.3)
- moved J2 0.27 mm to (0.00, 49.5)
- moved U$6 0.27 mm to (30.0, 94.0)
- moved IC2 0.27 mm to (50.5, 72.4)
- moved J1 0.25 mm to (0.00, 49.5)
Routing:
- net GND: track 2261.4 -> 2257.4 mm
- net VIN: track 83.3 -> 87.0 mm
- net +3V3: track 512.3 -> 511.3 mm
- net C28: track 146.0 -> 145.5 mm
- net TEMP_3: track 180.9 -> 180.4 mm
- net TEMP_2: track 172.8 -> 172.3 mm
- net TEMP_1: track 175.1 -> 174.6 mm
- net PROBE_VERT_2_DOWN: track 155.9 -> 155.4 mm
- net PROBE_HOR_2_LEFT: track 167.1 -> 166.6 mm
- net I_3_H: track 169.0 -> 168.5 mm
- net I_2_L: track 175.1 -> 174.6 mm
- net I_2_H: track 160.6 -> 160.0 mm
- net I_1_L: track 166.7 -> 166.2 mm
- net I_1_H: track 169.0 -> 168.5 mm
- net GND_TEMP: track 167.7 -> 167.2 mm
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Other:
- board text added: "GLOBAL ELECTRIC CIRCUIT DEBUG POWER SUPPLY BOARD REV 1.0 C. ANDERSON 7/30/19 NorthWest Research Associates DigiPen Institute of Technology"
- board text removed: "GLOBAL ELECTRIC CIRCUIT DEBUG POWER SUPPLY BOARD REV 1.0 C. ANDERSON 7/26/19 NorthWest Research Associates DigiPen Institute of Technology"
